File: assemble/assemble.kicad_pcb (KiCad board)
At the start: 2 copper layers, 110 parts, among them J1 Conn_02x04_Odd_Even, SW1 SW_Push, SW10 SW_Push, SW11 SW_Push, SW12 SW_Push, SW13 SW_Push, SW14 SW_Push, SW15 SW_Push, SW16 SW_Push, SW17 SW_Push, SW18 SW_Push, SW19 SW_Push, SW2 SW_Push, SW20 SW_Push, SW21 SW_Push, SW22 SW_Push, SW23 SW_Push, SW24 SW_Push, SW25 SW_Push, SW26 SW_Push, SW27 SW_Push, SW28 SW_Push, SW29 SW_Push, SW3 SW_Push, SW30 SW_Push, SW31 SW_Push, SW32 SW_Push, SW33 SW_Push, SW34 SW_Push, SW35 SW_Push, SW36 SW_Push, SW37 SW_Push, SW38 SW_Push, SW39 SW_Push, SW4 SW_Push, SW40 SW_Push, SW41 SW_Push, SW42 SW_Push, SW43 SW_SPDT, SW44 SW_SPDT, SW45 RotaryEncoder_Switch, SW5 SW_Push, SW6 SW_Push, SW7 SW_Push, SW8 SW_Push, SW9 SW_Push, U1 XIAO-nRF52840-SMD, U2 XIAO-nRF52840-SMD

Commit message: feat: implement PCB
Parts:
- added Ref**: Val**, kbd_Hole:m3_Screw_Hole_EdgeCuts, F.Cu at (67.0, 115.1)
- added Ref**: Val**, kbd_Hole:m2_Spacer_Hole_hex, F.Cu at (280.7, 119.1)
- added Ref**: Val**, kbd_Hole:m2_Spacer_Hole_hex, F.Cu at (280.7, 103.1)
- added Ref**: Val**, kbd_Hole:m3_Screw_Hole_EdgeCuts, F.Cu at (201.0, 39.0)
- added Ref**: Val**, kbd_Hole:m3_Screw_Hole_EdgeCuts, F.Cu at (42.0, 39.1)
- added Ref**: Val**, kbd_Hole:m3_Screw_Hole_EdgeCuts, F.Cu at (129.0, 39.0)
- added Ref**: Val**, kbd_Hole:m3_Screw_Hole_EdgeCuts, F.Cu at (129.0, 101.1)
- added Ref**: Val**, kbd_Hole:m3_Screw_Hole_EdgeCuts, F.Cu at (288.0, 39.0)
- added Ref**: Val**, kbd_Hole:m2_Spacer_Hole_hex, F.Cu at (254.7, 103.1)
- added Ref**: Val**, kbd_Hole:m3_Screw_Hole_EdgeCuts, F.Cu at (201.0, 101.1)
- added Ref**: Val**, kbd_Hole:m2_Spacer_Hole_hex, F.Cu at (254.7, 119.1)
- added Ref**: Val**, kbd_Hole:m3_Screw_Hole_EdgeCuts, F.Cu at (269.0, 95.0)
- moved D34 101.2 mm to (184.0, 70.0), turned to 90 degrees
- moved D26 98.3 mm to (187.0, 70.0), turned to 90 degrees
- moved D18 95.6 mm to (190.0, 70.0), turned to 90 degrees
- moved D10 93.0 mm to (193.0, 70.0), turned to 90 degrees
- moved AE-XCL102D333CR-G1 57.2 mm to (188.0, 101.0), turned to 180 degrees
- moved D5 43.8 mm to (254.0, 93.8), turned to 90 degrees
- moved U2 40.6 mm to (300.4, 108.0)
- moved D24 40.4 mm to (282.8, 79.7)
- moved SW16 40.4 mm to (262.1, 43.9)
- moved SW18 40.4 mm to (265.0, 77.0)
- moved SW24 40.4 mm to (248.4, 78.4)
- moved D14 40.4 mm to (299.1, 46.4)
- moved D16 40.4 mm to (299.2, 79.9)
- moved D22 40.4 mm to (282.9, 46.5)
- moved D23 40.4 mm to (282.6, 63.2)
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Other:
- board outline added: 292.2 x 101 mm

Commit message: feat: finish implement PCB
Parts:
- moved D30 20.0 mm to (241.0, 38.2)
- moved D31 20.0 mm to (242.9, 55.2)
- moved D6 20.0 mm to (236.7, 93.8)
- moved SW17 20.0 mm to (243.5, 60.4)
- moved AE-XCL102D333CR-G1 20.0 mm to (168.0, 101.0), turned to 0 degrees
- moved BT1 20.0 mm to (168.0, 41.0)
- moved D10 20.0 mm to (173.0, 70.0)
- moved D14 20.0 mm to (279.1, 46.4)
- moved D15 20.0 mm to (279.3, 63.2)
- moved D16 20.0 mm to (279.2, 79.9)
- moved D18 20.0 mm to (170.0, 70.0)
- moved D22 20.0 mm to (262.9, 46.5)
- moved D23 20.0 mm to (262.6, 63.2)
- moved D24 20.0 mm to (262.8, 79.7)
- moved D26 20.0 mm to (167.0, 70.0)
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Connections:
- U1 pad 3: BAT+L -> unconnected-(U1-P0.28_A2_D2-Pad3)
- U2 pad 1: BAT+R -> PIN1R
- U2 pad 18: PIN7R -> unconnected-(U2-NFC2-Pad18)
- U2 pad 2: PIN1R -> PIN2R
- U2 pad 4: PIN2R -> PIN3R
- U2 pad 5: PIN3R -> PIN4R
- U2 pad 6: PIN4R -> PIN5R
- U2 pad 7: PIN5R -> PIN6R
- U2 pad 8: PIN6R -> PIN7R
Routing:
- net Net-(D10-A): track 0.00 -> 239.4 mm, vias 0 -> 15
- net Net-(D26-A): track 0.00 -> 233.1 mm, vias 0 -> 14
- net Net-(D1-A): track 0.00 -> 230.4 mm, vias 0 -> 11
- net Net-(D25-A): track 0.00 -> 230.1 mm, vias 0 -> 15
- net Net-(D18-A): track 0.00 -> 228.2 mm, vias 0 -> 15
- net PIN2R: track 0.00 -> 226.4 mm, vias 0 -> 7
- net Net-(D17-A): track 0.00 -> 220.0 mm, vias 0 -> 11
- net PIN3R: track 0.00 -> 215.2 mm, vias 0 -> 9
- net PIN4R: track 0.00 -> 212.3 mm, vias 0 -> 7
- net PIN1R: track 0.00 -> 204.7 mm, vias 0 -> 5
- net Net-(AE-XCL102D333CR-G1-EN): track 0.00 -> 189.6 mm, vias 0 -> 1
- net Net-(SW43-B): track 0.00 -> 183.0 mm, vias 0 -> 1
- net Net-(AE-XCL102D333CR-G2-EN): track 0.00 -> 172.6 mm
- net Net-(SW44-B): track 0.00 -> 172.1 mm
- net Net-(D34-A): track 0.00 -> 167.7 mm, vias 0 -> 12
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Other:
- board size 292.2 x 101 mm -> 272.2 x 100.7 mm
- board text added: "ThingnusBall v1.0 designed by derui"

Commit message: fix: change position
Parts:
- moved Ref** 0.07 mm to (67.0, 115.0)
- moved Ref** 0.07 mm to (42.0, 39.0)
- moved Ref** 0.07 mm to (129.0, 101.0)
- moved Ref** 0.07 mm to (181.0, 101.0)
Other:
- outline, holes or cut-outs redrawn
Changed lines of the file:
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@@
 	(footprint "kbd_Hole:m3_Screw_Hole_EdgeCuts"
 		(layer "F.Cu")
-		(at 67 115.067739)
+		(at 67 115)
 		(descr "Mounting Hole 2.2mm, no annular, M2")
 		(tags "mounting hole 2.2mm no annular m2")
@@
 	(footprint "kbd_Hole:m3_Screw_Hole_EdgeCuts"
 		(layer "F.Cu")
-		(at 42 39.067739)
+		(at 42 39)
 		(descr "Mounting Hole 2.2mm, no annular, M2")
 		(tags "mounting hole 2.2mm no annular m2")
@@
 	(footprint "kbd_Hole:m3_Screw_Hole_EdgeCuts"
 		(layer "F.Cu")
-		(at 129 101.067739)
+		(at 129 101)
 		(descr "Mounting Hole 2.2mm, no annular, M2")
 		(tags "mounting hole 2.2mm no annular m2")
@@
 	(footprint "kbd_Hole:m3_Screw_Hole_EdgeCuts"
 		(layer "F.Cu")
-		(at 181 101.067739)
+		(at 181 101)
 		(descr "Mounting Hole 2.2mm, no annular, M2")
 		(tags "mounting hole 2.2mm no annular m2")
@@
 		(layer "Edge.Cuts")
 	)
-	(gr_arc
-		(start 19.802275 121)
-		(mid 19.094365 120.706303)
-		(end 18.802278 119.997727)
-		(stroke
-			(width 0.05)
-			(type default)
-		)
-		(layer "Edge.Cuts")
-	)
 	(gr_line
 		(start 256.3 105.5)
@@
 	(gr_line
 		(start 18.997732 33.997727)
-		(end 18.802278 119.997727)
+		(end 18.8 121)
 		(stroke
 			(width 0.05)
@@
 	)
 	(gr_line
-		(start 19.802275 121)
-		(end 107.736947 121)
+		(start 107.736947 121)
+		(end 18.8 121)
 		(stroke
 			(width 0.05)
@@
 	)
 	(segment
-		(start 161.2 36.4)
-		(end 161.2 35.401997)
+		(start 162.248943 35.199)
+		(end 278.261234 35.199)
 		(width 0.2)
 		(layer "F.Cu")
@@
 	)
 	(segment
-		(start 276.529334 35.4)
-		(end 278.462234 35.4)
+		(start 162.048943 34.999)
+		(end 162.248943 35.199)
 		(width 0.2)
 		(layer "F.Cu")
@@
 	)
 	(segment
-		(start 278.462234 35.4)
-		(end 282.067037 39.004803)
+		(start 161.2 35.401997)
+		(end 161.199 35.400997)
 		(width 0.2)
 		(layer "F.Cu")
@@
 	)
 	(segment
-		(start 162.248943 35.199)
-		(end 276.328334 35.199)
+		(start 278.261234 35.199)
+		(end 282.067037 39.004803)
 		(width 0.2)
 		(layer "F.Cu")
@@
 	)
 	(segment
-		(start 162.048943 34.999)
-		(end 162.248943 35.199)
+		(start 161.199 35.351057)
+		(end 161.551057 34.999)
 		(width 0.2)
 		(layer "F.Cu")
@@
 	)
 	(segment
-		(start 161.199 35.400997)
-		(end 161.199 35.351057)
+		(start 161.2 36.4)
+		(end 161.2 35.401997)
 		(width 0.2)
 		(layer "F.Cu")
@@
 	)
 	(segment
-		(start 161.2 35.401997)
-		(end 161.199 35.400997)
-		(width 0.2)
-		(layer "F.Cu")
-		(net 4)
-	)
-	(segment
-		(start 276.328334 35.199)
-		(end 276.529334 35.4)
-		(width 0.2)
-		(layer "F.Cu")
-		(net 4)
-	)
-	(segment
-		(start 161.199 35.351057)
-		(end 161.551057 34.999)
+		(start 161.199 35.400997)
+		(end 161.199 35.351057)
 		(width 0.2)
 		(layer "F.Cu")

Commit message: feat: change case and re-wired
Parts:
- Ref** (x4): footprint kbd_Hole:m2_Spacer_Hole_hex -> kbd_Hole:m2_Screw_Hole_EdgeCuts
- U1, U2: moved to B.Cu
- turned U1 to -90 degrees
- turned U2 to 90 degrees
Connections:
- AE-XCL102D333CR-G1 pad 6: Net-(BT1-+) -> B+R
- AE-XCL102D333CR-G2 pad 6: Net-(BT2-+) -> B+L
- BT1 pad 1: Net-(BT1-+) -> B+R
- BT2 pad 1: Net-(BT2-+) -> B+L
- U1 pad 3: unconnected-(U1-P0.28_A2_D2-Pad3) -> B+L
- U2 pad 18: unconnected-(U2-NFC2-Pad18) -> PIN7R
- U2 pad 3: INTR_R -> B+R
- U2 pad 4: PIN3R -> INTR_R
- U2 pad 5: PIN4R -> PIN3R
- U2 pad 6: PIN5R -> PIN4R
- U2 pad 7: PIN6R -> PIN5R
- U2 pad 8: PIN7R -> PIN6R
Routing:
- net B+L: track 0.00 -> 281.0 mm, vias 0 -> 5
- net B+R: track 0.00 -> 193.4 mm, vias 0 -> 5
- net Net-(BT1-+): track 59.1 -> 0.00 mm
- net Net-(BT2-+): track 59.1 -> 0.00 mm
- net INTR_R: track 59.5 -> 104.3 mm, vias 5 -> 6
- net Net-(D10-A): track 239.4 -> 205.7 mm, vias 15 -> 16
- net BAT-L: track 143.8 -> 173.2 mm, vias 0 -> 4
- net BAT+L: track 128.7 -> 157.9 mm, vias 0 -> 4
- net PIN1L: track 113.9 -> 94.9 mm, vias 5 -> 12
- net MISO: track 20.8 -> 38.8 mm, vias 0 -> 4
- net PIN5R: track 126.2 -> 144.1 mm, vias 7 -> 10
- net Net-(D25-A): track 230.1 -> 212.3 mm, vias 15 -> 20
- net PIN6L: track 167.6 -> 152.9 mm, vias 9 -> 10
- net PIN7R: track 135.4 -> 121.4 mm
- net Net-(D34-A): track 167.7 -> 154.4 mm
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Other:
- outline, holes or cut-outs redrawn

Commit message: fix: case problems
Parts:
- added Ref**: Val**, kbd_Hole:Mouse_Bite_Hole, F.Cu at (151.5, 69.5)
- added Ref**: Val**, kbd_Hole:Mouse_Bite_Hole, F.Cu at (155.4, 47.6)
- added Ref**: Val**, kbd_Hole:Mouse_Bite_Hole, F.Cu at (155.4, 43.1)
- added Ref**: Val**, kbd_Hole:Mouse_Bite_Hole, F.Cu at (155.4, 65.1)
- added Ref**: Val**, kbd_Hole:Mouse_Bite_Hole, F.Cu at (151.5, 60.5)
- added Ref**: Val**, kbd_Hole:Mouse_Bite_Hole, F.Cu at (155.4, 86.2)
- added Ref**: Val**, kbd_Hole:Mouse_Bite_Hole, F.Cu at (151.5, 43.0)
- added Ref**: Val**, kbd_Hole:Mouse_Bite_Hole, F.Cu at (151.5, 47.5)
- added Ref**: Val**, kbd_Hole:Mouse_Bite_Hole, F.Cu at (151.5, 95.1)
- added Ref**: Val**, kbd_Hole:Mouse_Bite_Hole, F.Cu at (155.4, 90.7)
- added Ref**: Val**, kbd_Hole:Mouse_Bite_Hole, F.Cu at (155.4, 60.6)
- added Ref**: Val**, kbd_Hole:Mouse_Bite_Hole, F.Cu at (155.4, 38.6)
- added Ref**: Val**, kbd_Hole:Mouse_Bite_Hole, F.Cu at (155.4, 69.6)
- added Ref**: Val**, kbd_Hole:Mouse_Bite_Hole, F.Cu at (151.5, 86.1)
- added Ref**: Val**, kbd_Hole:Mouse_Bite_Hole, F.Cu at (155.4, 95.2)
- added Ref**: Val**, kbd_Hole:Mouse_Bite_Hole, F.Cu at (151.5, 38.5)
- added Ref**: Val**, kbd_Hole:Mouse_Bite_Hole, F.Cu at (151.5, 90.6)
- added Ref**: Val**, kbd_Hole:Mouse_Bite_Hole, F.Cu at (151.5, 65.0)
- moved AE-XCL102D333CR-G1 3.00 mm to (165.0, 101.0)
- moved BT1 3.00 mm to (165.0, 41.0)
- moved D10 3.00 mm to (170.0, 70.0)
- moved D14 3.00 mm to (276.1, 46.4)
- moved D15 3.00 mm to (276.3, 63.2)
- moved D16 3.00 mm to (276.2, 79.9)
- moved D18 3.00 mm to (167.0, 70.0)
- moved D22 3.00 mm to (259.9, 46.5)
- moved D23 3.00 mm to (259.6, 63.2)
- moved D24 3.00 mm to (259.8, 79.7)
- moved D26 3.00 mm to (164.0, 70.0)
- moved D30 3.00 mm to (238.0, 38.2)
- moved D31 3.00 mm to (239.9, 55.2)
- moved D32 3.00 mm to (241.1, 71.6)
- moved D34 3.00 mm to (161.0, 70.0)
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Other:
- board size 272.2 x 100.7 mm -> 269.2 x 100.7 mm
